File: fcp-control-pcb/current_sensing.kicad_sch (KiCad schematic)
At the start: 3 parts

Commit message: pcb sans design review
Parts:
- removed U?: TLI4971-A050T5-U-E0001, Package_SON:Infineon_PG-TISON-8-5, symbol TLI4971-A050T5-U-E0001:TLI4971-A050T5-U-E0001
- added IC1: (no value), symbol Custom:L01Z050S05
- J9: renamed from J?; value (none) -> Current_Mode; footprint (none) -> Connector_PinHeader_2.54mm:PinHeader_1x02_P2.54mm_Vertical
- gave numbers to parts that had none: 1
Connections:
- net GND: now also IC1.2 (GND)
- net MOTOR_CURRENT: now also IC1.1 (VOUT)
- new net 5V: IC1.3 (+VCC_(+5V))
- no-connect marks 4 -> 2
Changed lines of the file:
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@@
 (kicad_sch (version 20211123) (generator eeschema)
   (paper "A4")
-  (junction (at 142.24 111.76) (diameter 0) (color 0 0 0 0)
-  )
   (junction (at 106.68 121.92) (diameter 0) (color 0 0 0 0)
   )
-  (junction (at 139.7 121.92) (diameter 0) (color 0 0 0 0)
-  )
   (no_connect (at 121.92 97.79))
-  (no_connect (at 186.69 97.79))
-  (no_connect (at 190.5 97.79))
   (no_connect (at 118.11 97.79))
-  (wire (pts (xy 171.45 97.79) (xy 171.45 100.33))
-    (stroke (width 0) (type default) (color 0 0 0 0))
-  )
-  (wire (pts (xy 179.07 111.76) (xy 142.24 111.76))
-    (stroke (width 0) (type default) (color 0 0 0 0))
-  )
   (wire (pts (xy 139.7 102.87) (xy 139.7 121.92))
     (stroke (width 0) (type default) (color 0 0 0 0))
@@
     (stroke (width 0) (type default) (color 0 0 0 0))
   )
-  (wire (pts (xy 175.26 97.79) (xy 175.26 121.92))
-    (stroke (width 0) (type default) (color 0 0 0 0))
-  )
   (wire (pts (xy 142.24 111.76) (xy 110.49 111.76))
     (stroke (width 0) (type default) (color 0 0 0 0))
   )
-  (wire (pts (xy 139.7 121.92) (xy 175.26 121.92))
-    (stroke (width 0) (type default) (color 0 0 0 0))
-  )
   (wire (pts (xy 102.87 97.79) (xy 102.87 100.33))
-    (stroke (width 0) (type default) (color 0 0 0 0))
-  )
-  (wire (pts (xy 182.88 102.87) (xy 182.88 97.79))
     (stroke (width 0) (type default) (color 0 0 0 0))
   )
@@
     (stroke (width 0) (type default) (color 0 0 0 0))
   )
-  (wire (pts (xy 179.07 97.79) (xy 179.07 111.76))
-    (stroke (width 0) (type default) (color 0 0 0 0))
-  )
   (hierarchical_label "FC_OUT" (shape output) (at 127 78.74 0)
     (effects (font (size 1.27 1.27)) (justify left))
   )
-  (hierarchical_label "MOTOR_CURRENT" (shape output) (at 182.88 102.87 0)
+  (hierarchical_label "MOTOR_CURRENT" (shape output) (at 158.75 82.55 180)
+    (effects (font (size 1.27 1.27)) (justify right))
+  )
+  (hierarchical_label "5V" (shape input) (at 194.31 82.55 0)
     (effects (font (size 1.27 1.27)) (justify left))
   )
-  (hierarchical_label "3.3V" (shape input) (at 171.45 100.33 270)
+  (hierarchical_label "GND" (shape input) (at 158.75 85.09 270)
     (effects (font (size 1.27 1.27)) (justify right))
   )
@@
     (effects (font (size 1.27 1.27)) (justify right))
   )
-  (hierarchical_label "CAP_OUT" (shape output) (at 195.58 78.74 0)
-    (effects (font (size 1.27 1.27)) (justify left))
-  )
   (hierarchical_label "3.3V" (shape input) (at 102.87 100.33 270)
     (effects (font (size 1.27 1.27)) (justify right))
@@
     (effects (font (size 1.27 1.27)) (justify right))
   )
-  (hierarchical_label "CAP_IN" (shape input) (at 167.64 78.74 180)
-    (effects (font (size 1.27 1.27)) (justify right))
-  )
-  (symbol (lib_id "TLI4971-A050T5-U-E0001:TLI4971-A050T5-U-E0001") (at 181.61 83.82 0) (unit 1)
-    (in_bom yes) (on_board yes) (fields_autoplaced)
-    (property "Reference" "U?" (id 0) (at 181.61 68.58 0))
-    (property "Value" "TLI4971-A050T5-U-E0001" (id 1) (at 181.61 71.12 0))
-    (property "Footprint" "Package_SON:Infineon_PG-TISON-8-5" (id 2) (at 182.88 76.2 0)
-      (effects (font (size 1.27 1.27)) hide)
-    )
-    (property "Datasheet" "https://www.infineon.com/dgdl/Infineon-TLI4971_25_50_75_120-DataSheet-v01_20-EN.pdf?fileId=5546d462700c0ae6017034d731621b09" (id 3) (at 182.88 76.2 0)
-      (effects (font (size 1.27 1.27)) hide)
-    )
-    (pin "1")
-    (pin "2")
-    (pin "3")
-    (pin "4")
-    (pin "5")
-    (pin "6")
-    (pin "7")
-    (pin "8")
-  )
   (symbol (lib_id "TLI4971-A050T5-U-E0001:TLI4971-A050T5-U-E0001") (at 113.03 83.82 0) (unit 1)
     (in_bom yes) (on_board yes) (fields_autoplaced)
-    (property "Reference" "U?" (id 0) (at 113.03 68.58 0))
+    (property "Reference" "U3" (id 0) (at 113.03 68.58 0))
     (property "Value" "TLI4971-A050T5-U-E0001" (id 1) (at 113.03 71.12 0))
     (property "Footprint" "Package_SON:Infineon_PG-TISON-8-5" (id 2) (at 114.3 76.2 0)
@@
     (pin "8")
   )
+  (symbol (lib_id "Custom:L01Z050S05") (at 158.75 82.55 0) (unit 1)
+    (in_bom yes) (on_board yes) (fields_autoplaced)
+    (property "Reference" "IC1" (id 0) (at 176.53 74.93 0))
+    (property "Value" "" (id 1) (at 176.53 77.47 0))
+    (property "Footprint" "" (id 2) (at 190.5 80.01 0)
+      (effects (font (size 1.27 1.27)) (justify left) hide)
+    )
+    (property "Datasheet" "https://www.mouser.com/datasheet/2/397/L01ZXXXS05-274998.pdf" (id 3) (at 190.5 82.55 0)
+      (effects (font (size 1.27 1.27)) (justify left) hide)
+    )
+    (property "Description" "Board Mount Current Sensors CURRENT SENSOR ( 50A; +5V)" (id 4) (at 190.5 85.09 0)
+      (effects (font (size 1.27 1.27)) (justify left) hide)
+    )
+    (property "Height" "" (id 5) (at 190.5 87.63 0)
+      (effects (font (size 1.27 1.27)) (justify left) hide)
+    )
+    (property "Manufacturer_Name" "Tamura" (id 6) (at 190.5 90.17 0)
+      (effects (font (size 1.27 1.27)) (justify left) hide)
+    )
+    (property "Manufacturer_Part_Number" "L01Z050S05" (id 7) (at 190.5 92.71 0)
+      (effects (font (size 1.27 1.27)) (justify left) hide)
+    )
+    (property "Mouser Part Number" "838-L01Z050S05" (id 8) (at 190.5 95.25 0)
+      (effects (font (size 1.27 1.27)) (justify left) hide)
+    )
+    (property "Mouser Price/Stock" "https://www.mouser.co.uk/ProductDetail/Tamura/L01Z050S05?qs=UO2oIyMggj%252Bpy1oyw7hC2g%3D%3D" (id 9) (at 190.5 97.79 0)
+      (effects (font (size 1.27 1.27)) (justify left) hide)
+    )
+    (property "Arrow Part Number" "" (id 10) (at 190.5 100.33 0)
+      (effects (font (size 1.27 1.27)) (justify left) hide)
+    )
+    (property "Arrow Price/Stock" "" (id 11) (at 190.5 102.87 0)
+      (effects (font (size 1.27 1.27)) (justify left) hide)
+    )
+    (property "Mouser Testing Part Number" "" (id 12) (at 190.5 105.41 0)
+      (effects (font (size 1.27 1.27)) (justify left) hide)
+    )
+    (property "Mouser Testing Price/Stock" "" (id 13) (at 190.5 107.95 0)
+      (effects (font (size 1.27 1.27)) (justify left) hide)
+    )
+    (pin "1")
+    (pin "2")
+    (pin "3")
+  )
   (symbol (lib_id "Connector:Conn_01x02_Male") (at 142.24 97.79 270) (unit 1)
     (in_bom yes) (on_board yes) (fields_autoplaced)
-    (property "Reference" "J?" (id 0) (at 143.51 97.1549 90)
+    (property "Reference" "J9" (id 0) (at 143.51 97.1549 90)
       (effects (font (size 1.27 1.27)) (justify left))
     )
-    (property "Value" "" (id 1) (at 143.51 99.6949 90)
+    (property "Value" "Current_Mode" (id 1) (at 143.51 99.6949 90)
       (effects (font (size 1.27 1.27)) (justify left))
     )
-    (property "Footprint" "" (id 2) (at 142.24 97.79 0)
+    (property "Footprint" "Connector_PinHeader_2.54mm:PinHeader_1x02_P2.54mm_Vertical" (id 2) (at 142.24 97.79 0)
       (effects (font (size 1.27 1.27)) hide)
     )
