File: fcp-control-pcb/switched_power.kicad_sch (KiCad schematic)
At the start: 10 parts

Commit message: pcb sans design review
Parts:
- added D9: LED, LED_SMD:LED_0603_1608Metric, symbol Device:LED
- added J12: OUT0, Connector_Molex:Molex_Mini-Fit_Jr_5569-02A2_2x01_P4.20mm_Horizontal, symbol Connector:Conn_01x02_Male
- added Q4: Q_NMOS_GDS, Package_TO_SOT_SMD:SOT-89-3_Handsoldering, symbol Device:Q_NMOS_GDS
- added R9: 1.5k, Resistor_SMD:R_0805_2012Metric_Pad1.20x1.40mm_HandSolder, symbol Device:R
- added TP16: OUT0, Connector_PinSocket_2.54mm:PinSocket_1x01_P2.54mm_Vertical, symbol Connector:TestPoint
- Q2: renamed from Q?; value (none) -> Q_NMOS_GDS; footprint (none) -> Package_TO_SOT_SMD:SOT-89-3_Handsoldering
- Q3: renamed from Q?; footprint (none) -> Package_TO_SOT_SMD:SOT-89-3_Handsoldering
- R7, R8: renamed from R?; footprint Resistor_SMD:R_0603_1608Metric -> Resistor_SMD:R_0805_2012Metric_Pad1.20x1.40mm_HandSolder
- gave numbers to parts that had none: 6
Connections:
- net GND: now also D9.1 (K), Q4.3 (S)
- net VCC: now also J12.1 (Pin_1)
- new net: J12.2 (Pin_2), Q4.2 (D), TP16.1
- new net: D9.2 (A), R9.1
- new net OUT0: Q4.1 (G), R9.2
