File: fcp-control-pcb/_autosave-voltage_sensing.kicad_sch (KiCad schematic)
At the start: 143 parts, among them J13 Conn_01x10_Male, J14 Conn_01x10_Male, J15 Conn_01x10_Male, U10 LM2902, U11 LM2902, U12 LM2902, U13 CD74HC4067SM, U14 CD74HC4067SM, U5 LM2902, U6 LM2902, U7 LM2902, U8 LM2902, U9 LM2902

Commit message: queen r1.1
Parts:
- removed C13, C14, C15, C16, C17, C18, C19, C20, C21, C22: 0.1 uF, Capacitor_SMD:C_0805_2012Metric_Pad1.18x1.45mm_HandSolder, symbol Device:C
- removed R10, R106, R107, R108, R109, R11, R110, R111, R112, R113, R114, R115, R116, R117, R12, R13, R14, R15, R16, R17, R18, R19, R20, R21, R22, R23, R24, R25, R42, R43, R44, R45, R46, R47, R48, R49, R50, R51, R52, R53, R54, R55, R56, R57, R74, R75, R76, R77, R78, R79, R80, R81, R82, R83, R84, R85, R86, R87, R88, R89: 20k, Resistor_SMD:R_0402_1005Metric_Pad0.72x0.64mm_HandSolder, symbol Device:R
- removed R100, R101, R102, R103, R104, R105, R118, R119, R120, R121, R122, R123, R124, R125, R126, R127, R128, R129, R26, R27, R28, R29, R30, R31, R32, R33, R34, R35, R36, R37, R38, R39, R40, R41, R58, R59, R60, R61, R62, R63, R64, R65, R66, R67, R68, R69, R70, R71, R72, R73, R90, R91, R92, R93, R94, R95, R96, R97, R98, R99: 91k, Resistor_SMD:R_0402_1005Metric_Pad0.72x0.64mm_HandSolder, symbol Device:R
- removed U10, U11, U12, U5, U6, U7, U8, U9: LM2902, Package_SO:SOIC-14_3.9x8.7mm_P1.27mm, symbol Amplifier_Operational:LM2902
- removed U13, U14: CD74HC4067SM, Package_SO:SSOP-24_5.3x8.2mm_P0.65mm, symbol 74xx:CD74HC4067SM
- added C15, C16: (no value), symbol Device:C_Small
- added J16: (no value), symbol Connector:Conn_01x02_Male
- added RN1, RN2, RN4: 3.3k, Package_SO:SOIC-16_4.55x10.3mm_P1.27mm, symbol Device:R_Pack08
- added RN3, RN7: (no value), symbol Device:R_Pack08
- added RN5, RN6, RN8: 1k, Package_SO:SOIC-16_4.55x10.3mm_P1.27mm, symbol Device:R_Pack08
- added U10, U8, U9: ADC1283, Package_SO:TSSOP-16_4.4x5mm_P0.65mm, symbol Custom:ADC1283
- added U6: (no value), symbol Custom:AS78L05RTR-G1
- added U7: (no value), symbol Custom:ADC1283
Connections:
- net +5V: now also U10.13 (DVCC), U7.13 (DVCC), U8.13 (DVCC), U9.13 (DVCC)
- net GND: now also C15.2, C16.2, RN5.1 (R1.1), RN5.2 (R2.1), RN5.3 (R3.1), RN5.4 (R4.1), RN5.5 (R5.1), RN5.6 (R6.1), RN5.7 (R7.1), RN5.8 (R8.1), RN6.1 (R1.1), RN6.2 (R2.1), RN6.3 (R3.1), RN6.4 (R4.1), RN6.5 (R5.1), RN6.6 (R6.1), RN6.7 (R7.1), RN6.8 (R8.1), RN7.10 (R7.2), RN7.11 (R6.2), RN7.12 (R5.2), RN7.13 (R4.2), RN7.14 (R3.2), RN7.15 (R2.2), RN7.16 (R1.2), RN7.9 (R8.2), RN8.1 (R1.1), RN8.2 (R2.1), RN8.3 (R3.1), RN8.4 (R4.1), RN8.5 (R5.1), RN8.6 (R6.1), RN8.7 (R7.1), RN8.8 (R8.1), U10.12 (DGND), U10.3 (AGND), U6.2 (GND), U7.12 (DGND), U7.3 (AGND), U8.12 (DGND), U8.3 (AGND), U9.12 (DGND), U9.3 (AGND)
- net VCC: now also C15.1, U6.3 (IN)
- net at J15.4 (Pin_4): now also RN4.14 (R3.2)
- net at J14.4 (Pin_4): now also RN1.16 (R1.2)
- net at J14.9 (Pin_9): now also RN2.13 (R4.2)
- net at J13.2 (Pin_2): now also RN2.16 (R1.2)
- net at J15.9 (Pin_9): now also RN1.11 (R6.2)
- net at J13.3 (Pin_3): now also RN3.8 (R8.1)
- net at J15.5 (Pin_5): now also RN4.15 (R2.2)
- net at J15.10 (Pin_10): now also RN1.12 (R5.2)
- net at J14.7 (Pin_7): now also RN2.11 (R6.2)
- net at J14.8 (Pin_8): now also RN2.12 (R5.2)
- net at J15.6 (Pin_6): now also RN4.16 (R1.2)
- net at J13.5 (Pin_5): now also RN3.6 (R6.1)
- net at J14.10 (Pin_10): now also RN2.14 (R3.2)
- net at J13.4 (Pin_4): now also RN3.7 (R7.1)
- net at J14.3 (Pin_3): now also RN1.15 (R2.2)
- net at J13.7 (Pin_7): now also RN3.4 (R4.1)
- net at J14.1 (Pin_1): now also RN1.13 (R4.2)
- net at J13.1 (Pin_1): now also RN2.15 (R2.2)
- net at J13.10 (Pin_10): now also RN3.1 (R1.1)
- net at J13.6 (Pin_6): now also RN3.5 (R5.1)
- net at J13.8 (Pin_8): now also RN3.3 (R3.1)
- net at J13.9 (Pin_9): now also RN3.2 (R2.1)
- net at J15.8 (Pin_8): now also RN1.10 (R7.2)
- net at J15.1 (Pin_1): now also RN4.11 (R6.2)
- net at J15.2 (Pin_2): now also RN4.12 (R5.2)
- net at J15.3 (Pin_3): now also RN4.13 (R4.2)
- net at J15.7 (Pin_7): now also RN1.9 (R8.2)
- net at J14.5 (Pin_5): now also RN2.9 (R8.2)
- net at J14.2 (Pin_2): now also RN1.14 (R3.2)
- net at J14.6 (Pin_6): now also RN2.10 (R7.2)
- new net: J16.2 (Pin_2), RN4.10 (R7.2)
- new net: J16.1 (Pin_1), RN4.9 (R8.2)
- new net +5VA: C16.1, U10.2 (AVCC), U6.1 (OUT), U7.2 (AVCC), U8.2 (AVCC), U9.2 (AVCC)
- new net ADCSelect0: U10.1 (CS)
- new net ADCSelect1: U9.1 (CS)
- new net ADCSelect2: U8.1 (CS)
- new net ADCSelect3: U7.1 (CS)
- new net DIN: U10.14 (DIN), U7.14 (DIN), U8.14 (DIN), U9.14 (DIN)
- new net DOUT: U10.15 (DOUT), U7.15 (DOUT), U8.15 (DOUT), U9.15 (DOUT)
- new net SCLK: U10.16 (SCLK), U7.16 (SCLK), U8.16 (SCLK), U9.16 (SCLK)
- new net cell1: RN3.16 (R1.2), RN7.1 (R1.1), U10.4 (IN0)
- new net cell10: RN2.2 (R2.1), RN6.15 (R2.2), U9.5 (IN1)
- new net cell11: RN2.3 (R3.1), RN6.14 (R3.2), U9.6 (IN2)
- new net cell12: RN2.4 (R4.1), RN6.13 (R4.2), U9.7 (IN3)
- new net cell13: RN2.5 (R5.1), RN6.12 (R5.2), U9.8 (IN4)
- new net cell14: RN2.6 (R6.1), RN6.11 (R6.2), U9.9 (IN5)
- new net cell15: RN2.7 (R7.1), RN6.10 (R7.2), U9.10 (IN6)
- new net cell16: RN2.8 (R8.1), RN6.9 (R8.2), U9.11 (IN7)
- new net cell17: RN1.1 (R1.1), RN5.16 (R1.2), U8.4 (IN0)
- new net cell18: RN1.2 (R2.1), RN5.15 (R2.2), U8.5 (IN1)
- new net cell19: RN1.3 (R3.1), RN5.14 (R3.2), U8.6 (IN2)
- new net cell2: RN3.15 (R2.2), RN7.2 (R2.1), U10.5 (IN1)
- new net cell20: RN1.4 (R4.1), RN5.13 (R4.2), U8.7 (IN3)
- new net cell21: RN1.5 (R5.1), RN5.12 (R5.2), U8.8 (IN4)
- new net cell22: RN1.6 (R6.1), RN5.11 (R6.2), U8.9 (IN5)
- new net cell23: RN1.7 (R7.1), RN5.10 (R7.2), U8.10 (IN6)
- new net cell24: RN1.8 (R8.1), RN5.9 (R8.2), U8.11 (IN7)
- new net cell25: RN4.1 (R1.1), RN8.16 (R1.2), U7.4 (IN0)
- new net cell26: RN4.2 (R2.1), RN8.15 (R2.2), U7.5 (IN1)
- new net cell27: RN4.3 (R3.1), RN8.14 (R3.2), U7.6 (IN2)
- new net cell28: RN4.4 (R4.1), RN8.13 (R4.2), U7.7 (IN3)
- new net cell29: RN4.5 (R5.1), RN8.12 (R5.2), U7.8 (IN4)
- new net cell3: RN3.14 (R3.2), RN7.3 (R3.1), U10.6 (IN2)
- new net cell30: RN4.6 (R6.1), RN8.11 (R6.2), U7.9 (IN5)
- new net cell4: RN3.13 (R4.2), RN7.4 (R4.1), U10.7 (IN3)
- new net cell5: RN3.12 (R5.2), RN7.5 (R5.1), U10.8 (IN4)
- new net cell6: RN3.11 (R6.2), RN7.6 (R6.1), U10.9 (IN5)
- new net cell7: RN3.10 (R7.2), RN7.7 (R7.1), U10.10 (IN6)
- new net cell8: RN3.9 (R8.2), RN7.8 (R8.1), U10.11 (IN7)
- new net cell9: RN2.1 (R1.1), RN6.16 (R1.2), U9.4 (IN0)
- new net extra1: RN4.7 (R7.1), RN8.10 (R7.2), U7.10 (IN6)
- new net extra2: RN4.8 (R8.1), RN8.9 (R8.2), U7.11 (IN7)
- no-connect marks 8 -> 0
Other:
- moved on the sheet: J13, J14, J15
