File: fcp-control-pcb/voltage_limiting.kicad_sch (KiCad schematic)
At the start: 15 parts

Commit message: pcb sans design review
Parts:
- removed D? (x2): DIODE, symbol Simulation_SPICE:DIODE
- added D3, D4: D, Diode_SMD:D_PowerDI-5, symbol Device:D
- C6: renamed from C?; footprint (none) -> Capacitor_SMD:C_0805_2012Metric_Pad1.18x1.45mm_HandSolder
- J8: renamed from J?; value (none) -> LimiterBypass; footprint Connector_Molex:Molex_Mini-Fit_Jr_5569-02A2_2x01_P4.20mm_Horizontal -> Connector_PinHeader_2.54mm:PinHeader_1x02_P2.54mm_Vertical
- Q1: renamed from Q?; value (none) -> AONR21321; footprint (none) -> custom:TRANS_AONR21321
- R1, R2: renamed from R?; footprint (none) -> Resistor_SMD:R_0805_2012Metric_Pad1.20x1.40mm_HandSolder
- RV1, RV2: renamed from RV?; footprint (none) -> custom:TRIM_3361P-1-203GLF
- TP10, TP11, TP12, TP13, TP9: renamed from TP?; footprint (none) -> TestPoint:TestPoint_Pad_4.0x4.0mm
- U2: renamed from U?; footprint SOIC127P599X175-8N -> custom:SOIC127P599X175-8N
Connections:
- net +5V: now also RV2.3; no longer RV2.1
- net CAP+: now also RV1.3, D3.1 (K), D4.2 (A); no longer J8.1 (Pin_1), RV1.1
- net CHRG+: now also D3.2 (A)
- net CHRG-: now also J8.1 (Pin_1), RV1.1, RV2.1; no longer RV1.3, RV2.3
- net DSCHRG+: now also D4.1 (K)
- net FC+: no longer J8.2 (Pin_2)
- net at Q1.4, R2.2, TP11.1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: now also J8.2 (Pin_2)
Other:
- moved on the sheet: J8

Commit message: queen r1.1
Parts:
- removed R2: 4.7k, Resistor_SMD:R_0805_2012Metric_Pad1.20x1.40mm_HandSolder, symbol Device:R
- added R?: 4.7k, Resistor_SMD:R_0805_2012Metric_Pad1.20x1.40mm_HandSolder, symbol Device:R
- added U?: (no value), symbol Driver_FET:ZXGD3003E6
Connections:
- net CHRG-: now also U?.3 (GND)
- net FC+: now also R?.1, U?.1 (VCC)
- net at J8.2 (Pin_2), TP11.1, U2.7 (OUT): now also R?.2, U?.2 (IN1), U?.5 (IN2); no longer Q1.4
- new net: Q1.4, U?.4 (SINK), U?.6 (SOURCE)
Other:
- moved on the sheet: Q1, TP12, TP13

Commit message: Fixed autosave issues
Parts:
- U5: renamed from U?; value (none) -> ZXGD3003E6; footprint (none) -> Package_TO_SOT_SMD:SOT-23-6
- gave numbers to parts that had none: 1
Changed lines of the file:
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@@
   (symbol (lib_id "Driver_FET:ZXGD3003E6") (at 182.88 96.52 0) (unit 1)
     (in_bom yes) (on_board yes) (fields_autoplaced)
-    (property "Reference" "U?" (id 0) (at 184.8994 86.36 0)
-      (effects (font (size 1.27 1.27)) (justify left))
-    )
-    (property "Value" "" (id 1) (at 184.8994 88.9 0)
-      (effects (font (size 1.27 1.27)) (justify left))
-    )
-    (property "Footprint" "" (id 2) (at 182.88 109.22 0)
+    (property "Reference" "U5" (id 0) (at 184.8994 86.36 0)
+      (effects (font (size 1.27 1.27)) (justify left))
+    )
+    (property "Value" "ZXGD3003E6" (id 1) (at 184.8994 88.9 0)
+      (effects (font (size 1.27 1.27)) (justify left))
+    )
+    (property "Footprint" "Package_TO_SOT_SMD:SOT-23-6" (id 2) (at 182.88 109.22 0)
       (effects (font (size 1.27 1.27)) hide)
     )
@@
   (symbol (lib_id "Device:R") (at 162.56 87.63 0) (unit 1)
     (in_bom yes) (on_board yes) (fields_autoplaced)
-    (property "Reference" "R?" (id 0) (at 165.1 86.3599 0)
-      (effects (font (size 1.27 1.27)) (justify left))
-    )
+    (property "Reference" "R2" (id 0) (at 165.1 86.3599 0)
+      (effects (font (size 1.27 1.27)) (justify left))
+    )
