File: fcp-control-pcb/fcp-control-pcb.kicad_sch (KiCad schematic)
At the start: 30 parts

Commit message: pcb sans design review
Parts:
- removed F?: (no value), symbol Device:Fuse
- removed F?: Fuse, symbol Device:Fuse
- removed J?: (no value), Connector_Molex:Molex_Mini-Fit_Jr_5569-02A2_2x01_P4.20mm_Horizontal, symbol Connector:Conn_01x02_Male
- removed TP? (x3): (no value), symbol Connector:TestPoint
- added D1, D2: D, custom:TSOT-23-3(2), symbol Device:D
- added TP17: GND, TestPoint:TestPoint_Pad_4.0x4.0mm, symbol Connector:TestPoint
- A1: renamed from A?; value (none) -> Arduino_Nano_Every; footprint (none) -> Module:Arduino_Nano
- C1, C2: renamed from C?; footprint Capacitor_SMD:C_0805_2012Metric -> Capacitor_SMD:C_0805_2012Metric_Pad1.18x1.45mm_HandSolder
- C3: renamed from C?; footprint Capacitor_SMD:C_0201_0603Metric -> Capacitor_SMD:C_0805_2012Metric_Pad1.18x1.45mm_HandSolder
- C4, C5: renamed from C?; footprint Capacitor_SMD:C_0603_1608Metric -> Capacitor_SMD:C_0805_2012Metric_Pad1.18x1.45mm_HandSolder
- F1: renamed from F?; footprint digikey-footprints:3586KTR -> custom:3586KTR
- J3: renamed from J?; value (none) -> CAPACITOR; footprint (none) -> custom:VP0265540000G
- J4: renamed from J?; value (none) -> FUELCELL; footprint (none) -> custom:VP0265540000G
- J6: renamed from J?; value (none) -> DISCHARGER
- J7: renamed from J?; value (none) -> CHARGER; footprint (none) -> Connector_Molex:Molex_Mini-Fit_Jr_5569-02A2_2x01_P4.20mm_Horizontal
- TP3: renamed from TP?; value (none) -> VCC; footprint (none) -> TestPoint:TestPoint_Pad_4.0x4.0mm
- TP4: renamed from TP?; value (none) -> FC_CURRENT; footprint (none) -> TestPoint:TestPoint_Pad_4.0x4.0mm
- TP5: renamed from TP?; value (none) -> MOTOR_CURRENT; footprint (none) -> TestPoint:TestPoint_Pad_4.0x4.0mm
- TP7: renamed from TP?; value (none) -> SAFETY_TX; footprint (none) -> TestPoint:TestPoint_Pad_4.0x4.0mm
- TP8: renamed from TP?; value (none) -> TLMTR_TX; footprint (none) -> TestPoint:TestPoint_Pad_4.0x4.0mm
- U1: renamed from U?; value (none) -> MAX15462AB; footprint (none) -> digikey-footprints:TDFN-8-1EP
- gave numbers to parts that had none: 7
Connections:
- net +5V: now also C3.1, L1.2, U1.4 (FB/Vout); no longer C2.1, U1.3 (Vcc)
- net CAP+: now also F1.2, J3.1 (Pin_1)
- net FC+: now also J4.1 (Pin_1), D2.2 (A)
- net GND: now also TP17.1
- net VCC: now also D1.2 (A)
- net VinNano: now also A1.30 (VIN)
- new net: C2.1, U1.3 (Vcc)
- new net Voltage Sensing/VCC: D1.1 (K), D2.1 (K)
- no-connect marks 1 -> 2
Other:
- sheet Pumps renamed Switched Power Out
- added sheet Voltage Sensing (voltage_sensing.kicad_sch)
- sheet Current Sensing ports: added 5V; removed CAP_IN, CAP_OUT
- sheet Switched Power Out ports: added OUT0; removed none
- moved on the sheet: TP3

Commit message: queen r1.1
Parts:
- removed D1, D2: D, custom:TSOT-23-3(2), symbol Device:D
- added C?: 0.33uF, symbol Device:C_Small
- added C?: 0.1uF, symbol Device:C_Small
- added U?: AS78L05RTR-G1, Package_TO_SOT_SMD:SOT-89-3_Handsoldering, symbol Custom:AS78L05RTR-G1
- J4: DigikeyPN (none) -> VP0265540000G-ND
- U1: value MAX15462AB -> (none); footprint digikey-footprints:TDFN-8-1EP -> (none)
Connections:
- net GND: now also C?.2, C?.2, U?.2 (GND)
- net VCC: now also C?.1, U?.3 (IN)
- net D3 renamed ADCSelect0
- net D4 renamed ADCSelect1
- net D5 renamed ADCSelect2
- net D6 renamed ADCSelect3
- new net +5VA: C?.1, U?.1 (OUT)
Other:
- sheet Voltage Sensing ports: added ADCSelect0, ADCSelect1, ADCSelect2, ADCSelect3, DIN, DOUT, SCLK; removed MUX0_OUT, MUX1_OUT, MUXSEL0, MUXSEL1, MUXSEL2, MUXSEL3, VCC
- note added: "5V Regulator"
- note added: "Alternative 5V Regulator"
- note removed: "5V LDO"

Commit message: Fixed autosave issues
Parts:
- added J5: ArduinoVCCPower, Connector_PinHeader_2.54mm:PinHeader_1x02_P2.54mm_Vertical, symbol Connector:Conn_01x02_Male
- C13, C14: renamed from C?; footprint (none) -> Capacitor_SMD:C_0805_2012Metric_Pad1.18x1.45mm_HandSolder
- C5: value 1uF -> 10uF
- U1: value (none) -> MAX15462AB; footprint (none) -> Package_DFN_QFN:TDFN-8-1EP_2x2mm_P0.5mm_EP0.8x1.2mm
- gave numbers to parts that had none: 1
Connections:
- net +5VA is gone; now on net +5V: C14.1, U4.1 (OUT)
- net D8 is gone; now on net BigPump: A1.11 (D8), J1.11 (Pin_11)
- net BigPump: no longer A1.12 (D9), J1.12 (Pin_12)
- net VCC: now also J5.2 (Pin_2)
- net VinNano: now also J5.1 (Pin_1)
- new net D9: A1.12 (D9), J1.12 (Pin_12)
