File: fcp-control-pcb/voltage_sensing.kicad_sch (KiCad schematic)
At the start: 19 parts, among them J13 Conn_01x10_Male, J14 Conn_01x10_Male, J15 Conn_01x10_Male, J16 ExtraAnalogs, U10 ADC1283, U6 AS78L05RTR-G1, U7 ADC1283, U8 ADC1283, U9 ADC1283

Commit message: Queen 1.1
Parts:
- added J17: (no value), symbol Connector:Conn_01x02_Male
Connections:
- net GND: no longer C15.2, C16.2, RN5.1 (R1.1), RN5.2 (R2.1), RN5.3 (R3.1), RN5.4 (R4.1), RN5.5 (R5.1), RN5.6 (R6.1), RN5.7 (R7.1), RN5.8 (R8.1), RN6.1 (R1.1), RN6.2 (R2.1), RN6.3 (R3.1), RN6.4 (R4.1), RN6.5 (R5.1), RN6.6 (R6.1), RN6.7 (R7.1), RN6.8 (R8.1), RN7.10 (R7.2), RN7.11 (R6.2), RN7.12 (R5.2), RN7.13 (R4.2), RN7.14 (R3.2), RN7.15 (R2.2), RN7.16 (R1.2), RN7.9 (R8.2), RN8.1 (R1.1), RN8.2 (R2.1), RN8.3 (R3.1), RN8.4 (R4.1), RN8.5 (R5.1), RN8.6 (R6.1), RN8.7 (R7.1), RN8.8 (R8.1), U10.3 (AGND), U6.2 (GND), U7.3 (AGND), U8.3 (AGND), U9.3 (AGND)
- net VCC renamed +12VA
- net +12VA: now also J17.1 (Pin_1)
- new net GNDA: C15.2, C16.2, J17.2 (Pin_2), RN5.1 (R1.1), RN5.2 (R2.1), RN5.3 (R3.1), RN5.4 (R4.1), RN5.5 (R5.1), RN5.6 (R6.1), RN5.7 (R7.1), RN5.8 (R8.1), RN6.1 (R1.1), RN6.2 (R2.1), RN6.3 (R3.1), RN6.4 (R4.1), RN6.5 (R5.1), RN6.6 (R6.1), RN6.7 (R7.1), RN6.8 (R8.1), RN7.10 (R7.2), RN7.11 (R6.2), RN7.12 (R5.2), RN7.13 (R4.2), RN7.14 (R3.2), RN7.15 (R2.2), RN7.16 (R1.2), RN7.9 (R8.2), RN8.1 (R1.1), RN8.2 (R2.1), RN8.3 (R3.1), RN8.4 (R4.1), RN8.5 (R5.1), RN8.6 (R6.1), RN8.7 (R7.1), RN8.8 (R8.1), U10.3 (AGND), U6.2 (GND), U7.3 (AGND), U8.3 (AGND), U9.3 (AGND)
Changed lines of the file:
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@@
   (junction (at 422.91 198.12) (diameter 0) (color 0 0 0 0)
   )
-  (junction (at 340.36 299.72) (diameter 0) (color 0 0 0 0)
-  )
   (junction (at 243.84 194.31) (diameter 0) (color 0 0 0 0)
   )
@@
   (junction (at 247.65 153.67) (diameter 0) (color 0 0 0 0)
   )
-  (junction (at 383.54 299.72) (diameter 0) (color 0 0 0 0)
-  )
   (junction (at 243.84 252.73) (diameter 0) (color 0 0 0 0)
   )
@@
   (junction (at 254 290.83) (diameter 0) (color 0 0 0 0)
   )
+  (junction (at 304.8 299.72) (diameter 0) (color 0 0 0 0)
+  )
   (junction (at 250.19 175.26) (diameter 0) (color 0 0 0 0)
   )
@@
     (stroke (width 0) (type default) (color 0 0 0 0))
   )
+  (wire (pts (xy 186.69 104.14) (xy 186.69 106.68))
+    (stroke (width 0) (type default) (color 0 0 0 0))
+  )
   (wire (pts (xy 242.57 158.75) (xy 257.81 158.75))
     (stroke (width 0) (type default) (color 0 0 0 0))
@@
     (stroke (width 0) (type default) (color 0 0 0 0))
   )
+  (wire (pts (xy 181.61 104.14) (xy 186.69 104.14))
+    (stroke (width 0) (type default) (color 0 0 0 0))
+  )
   (wire (pts (xy 340.36 195.58) (xy 340.36 157.48))
     (stroke (width 0) (type default) (color 0 0 0 0))
@@
     (stroke (width 0) (type default) (color 0 0 0 0))
   )
+  (wire (pts (xy 186.69 101.6) (xy 186.69 97.79))
+    (stroke (width 0) (type default) (color 0 0 0 0))
+  )
   (wire (pts (xy 422.91 198.12) (xy 422.91 236.22))
     (stroke (width 0) (type default) (color 0 0 0 0))
@@
     (stroke (width 0) (type default) (color 0 0 0 0))
   )
-  (wire (pts (xy 426.72 299.72) (xy 383.54 299.72))
-    (stroke (width 0) (type default) (color 0 0 0 0))
-  )
   (wire (pts (xy 344.17 193.04) (xy 344.17 154.94))
     (stroke (width 0) (type default) (color 0 0 0 0))
@@
     (stroke (width 0) (type default) (color 0 0 0 0))
   )
-  (wire (pts (xy 340.36 299.72) (xy 269.24 299.72))
+  (wire (pts (xy 340.36 299.72) (xy 304.8 299.72))
     (stroke (width 0) (type default) (color 0 0 0 0))
   )
@@
     (stroke (width 0) (type default) (color 0 0 0 0))
   )
+  (wire (pts (xy 181.61 101.6) (xy 186.69 101.6))
+    (stroke (width 0) (type default) (color 0 0 0 0))
+  )
   (wire (pts (xy 179.07 199.39) (xy 214.63 199.39))
     (stroke (width 0) (type default) (color 0 0 0 0))
@@
     (stroke (width 0) (type default) (color 0 0 0 0))
   )
-  (wire (pts (xy 340.36 299.72) (xy 383.54 299.72))
-    (stroke (width 0) (type default) (color 0 0 0 0))
-  )
   (wire (pts (xy 238.76 276.86) (xy 256.54 276.86))
     (stroke (width 0) (type default) (color 0 0 0 0))
@@
   )
   (wire (pts (xy 184.15 276.86) (xy 224.79 276.86))
+    (stroke (width 0) (type default) (color 0 0 0 0))
+  )
+  (wire (pts (xy 304.8 299.72) (xy 269.24 299.72))
     (stroke (width 0) (type default) (color 0 0 0 0))
   )
@@
     (pin "9")
   )
+  (symbol (lib_id "power:GNDA") (at 304.8 299.72 0) (unit 1)
+    (in_bom yes) (on_board yes) (fields_autoplaced)
+    (property "Reference" "#PWR0136" (id 0) (at 304.8 306.07 0)
+      (effects (font (size 1.27 1.27)) hide)
+    )
+    (property "Value" "GNDA" (id 1) (at 304.8 304.8 0))
+    (property "Footprint" "" (id 2) (at 304.8 299.72 0)
+      (effects (font (size 1.27 1.27)) hide)
+    )
+    (property "Datasheet" "" (id 3) (at 304.8 299.72 0)
+      (effects (font (size 1.27 1.27)) hide)
+    )
+    (pin "1")
+  )
   (symbol (lib_id "power:+5V") (at 422.91 140.97 0) (unit 1)
     (in_bom yes) (on_board yes) (fields_autoplaced)
@@
     (pin "2")
     (pin "3")
+  )
+  (symbol (lib_id "power:GNDA") (at 294.64 123.19 0) (unit 1)
+    (in_bom yes) (on_board yes) (fields_autoplaced)
+    (property "Reference" "#PWR0135" (id 0) (at 294.64 129.54 0)
+      (effects (font (size 1.27 1.27)) hide)
+    )
+    (property "Value" "GNDA" (id 1) (at 294.64 128.27 0))
+    (property "Footprint" "" (id 2) (at 294.64 123.19 0)
+      (effects (font (size 1.27 1.27)) hide)
+    )
+    (property "Datasheet" "" (id 3) (at 294.64 123.19 0)
+      (effects (font (size 1.27 1.27)) hide)
+    )
+    (pin "1")
   )
   (symbol (lib_id "Connector:Conn_01x10_Male") (at 173.99 237.49 0) (unit 1)
@@
     (pin "9")
   )
-  (symbol (lib_id "power:GND") (at 383.54 299.72 0) (unit 1)
-    (in_bom yes) (on_board yes) (fields_autoplaced)
-    (property "Reference" "#PWR0127" (id 0) (at 383.54 306.07 0)
-      (effects (font (size 1.27 1.27)) hide)
-    )
-    (property "Value" "GND" (id 1) (at 383.54 304.8 0))
-    (property "Footprint" "" (id 2) (at 383.54 299.72 0)
-      (effects (font (size 1.27 1.27)) hide)
-    )
-    (property "Datasheet" "" (id 3) (at 383.54 299.72 0)
-      (effects (font (size 1.27 1.27)) hide)
-    )
-    (pin "1")
-  )
-  (symbol (lib_id "power:VCC") (at 269.24 110.49 0) (unit 1)
-    (in_bom yes) (on_board yes) (fields_autoplaced)
-    (property "Reference" "#PWR0129" (id 0) (at 269.24 114.3 0)
-      (effects (font (size 1.27 1.27)) hide)
-    )
-    (property "Value" "VCC" (id 1) (at 269.24 105.41 0))
-    (property "Footprint" "" (id 2) (at 269.24 110.49 0)
-      (effects (font (size 1.27 1.27)) hide)
-    )
-    (property "Datasheet" "" (id 3) (at 269.24 110.49 0)
-      (effects (font (size 1.27 1.27)) hide)
-    )
-    (pin "1")
+  (symbol (lib_id "power:GND") (at 426.72 299.72 0) (unit 1)
+    (in_bom yes) (on_board yes) (fields_autoplaced)
+    (property "Reference" "#PWR0127" (id 0) (at 426.72 306.07 0)
+      (effects (font (size 1.27 1.27)) hide)
+    )
+    (property "Value" "GND" (id 1) (at 426.72 304.8 0))
+    (property "Footprint" "" (id 2) (at 426.72 299.72 0)
+      (effects (font (size 1.27 1.27)) hide)
+    )
+    (property "Datasheet" "" (id 3) (at 426.72 299.72 0)
+      (effects (font (size 1.27 1.27)) hide)
+    )
+    (pin "1")
+  )
+  (symbol (lib_id "power:GNDA") (at 186.69 106.68 0) (unit 1)
+    (in_bom yes) (on_board yes) (fields_autoplaced)
+    (property "Reference" "#PWR0129" (id 0) (at 186.69 113.03 0)
+      (effects (font (size 1.27 1.27)) hide)
+    )
+    (property "Value" "" (id 1) (at 186.69 111.76 0))
+    (property "Footprint" "" (id 2) (at 186.69 106.68 0)
+      (effects (font (size 1.27 1.27)) hide)
+    )
+    (property "Datasheet" "" (id 3) (at 186.69 106.68 0)
+      (effects (font (size 1.27 1.27)) hide)
+    )
+    (pin "1")
+  )
+  (symbol (lib_id "Connector:Conn_01x02_Male") (at 176.53 101.6 0) (unit 1)
+    (in_bom yes) (on_board yes)
+    (property "Reference" "J17" (id 0) (at 179.2732 97.0026 0))
+    (property "Value" "" (id 1) (at 179.2732 99.314 0))
+    (property "Footprint" "" (id 2) (at 176.53 101.6 0)
+      (effects (font (size 1.27 1.27)) hide)
+    )
+    (property "Datasheet" "https://www.molex.com/pdm_docs/ps/PS-5556-001.pdf" (id 3) (at 176.53 101.6 0)
+      (effects (font (size 1.27 1.27)) hide)
+    )
+    (property "DigikeyPN" "0050361758-ND" (id 4) (at 176.53 101.6 0)
+      (effects (font (size 1.27 1.27)) hide)
+    )
+    (pin "1")
+    (pin "2")
   )
   (symbol (lib_id "Device:R_Pack08") (at 231.14 153.67 90) (unit 1)
@@
     (pin "9")
   )
-  (symbol (lib_id "power:GND") (at 294.64 123.19 0) (unit 1)
-    (in_bom yes) (on_board yes) (fields_autoplaced)
-    (property "Reference" "#PWR0130" (id 0) (at 294.64 129.54 0)
-      (effects (font (size 1.27 1.27)) hide)
-    )
-    (property "Value" "GND" (id 1) (at 294.64 128.27 0))
-    (property "Footprint" "" (id 2) (at 294.64 123.19 0)
-      (effects (font (size 1.27 1.27)) hide)
-    )
-    (property "Datasheet" "" (id 3) (at 294.64 123.19 0)
-      (effects (font (size 1.27 1.27)) hide)
-    )
-    (pin "1")
-  )
   (symbol (lib_id "Device:C_Small") (at 278.13 115.57 0) (unit 1)
     (in_bom yes) (on_board yes) (fields_autoplaced)
@@
     (pin "1")
     (pin "2")
+  )
+  (symbol (lib_id "power:+12VA") (at 186.69 97.79 0) (unit 1)
+    (in_bom yes) (on_board yes) (fields_autoplaced)
+    (property "Reference" "#PWR0130" (id 0) (at 186.69 101.6 0)
+      (effects (font (size 1.27 1.27)) hide)
+    )
+    (property "Value" "" (id 1) (at 186.69 92.71 0))
+    (property "Footprint" "" (id 2) (at 186.69 97.79 0)
+      (effects (font (size 1.27 1.27)) hide)
+    )
+    (property "Datasheet" "" (id 3) (at 186.69 97.79 0)
+      (effects (font (size 1.27 1.27)) hide)
+    )
+    (pin "1")
   )
   (symbol (lib_id "Device:R_Pack08") (at 229.87 269.24 270) (mirror x) (unit 1)
@@
     (pin "9")
   )
+  (symbol (lib_id "power:+12VA") (at 269.24 110.49 0) (unit 1)
+    (in_bom yes) (on_board yes) (fields_autoplaced)
+    (property "Reference" "#PWR0134" (id 0) (at 269.24 114.3 0)
+      (effects (font (size 1.27 1.27)) hide)
+    )
+    (property "Value" "+12VA" (id 1) (at 269.24 105.41 0))
+    (property "Footprint" "" (id 2) (at 269.24 110.49 0)
+      (effects (font (size 1.27 1.27)) hide)
+    )
+    (property "Datasheet" "" (id 3) (at 269.24 110.49 0)
+      (effects (font (size 1.27 1.27)) hide)
+    )
+    (pin "1")
+  )
   (symbol (lib_id "Connector:Conn_01x02_Male") (at 215.9 146.05 0) (unit 1)
